File: KiCad/17B06E-Macropad.kicad_sch (KiCad schematic)
At the start: 64 parts, among them SW1 RotaryEncoder_Switch, SW2 RotaryEncoder_Switch, SW3 RotaryEncoder_Switch, SW4 RotaryEncoder_Switch, SW5 RotaryEncoder_Switch, SW6 RotaryEncoder_Switch

Commit message: update
Parts:
- OLED1: I2C (none) -> I²C1
Connections:
- net VBUS renamed VCC +5V
- net VCC +5V: now also LED1.1 (VDD), LED10.1 (VDD), LED11.1 (VDD), LED12.1 (VDD), LED13.1 (VDD), LED14.1 (VDD), LED15.1 (VDD), LED16.1 (VDD), LED2.1 (VDD), LED3.1 (VDD), LED4.1 (VDD), LED5.1 (VDD), LED6.1 (VDD), LED7.1 (VDD), LED8.1 (VDD), LED9.1 (VDD), OLED1.2 (Pin_2)
- removed net VCC: A1.35 (ADC_VREF), LED1.1 (VDD), LED10.1 (VDD), LED11.1 (VDD), LED12.1 (VDD), LED13.1 (VDD), LED14.1 (VDD), LED15.1 (VDD), LED16.1 (VDD), LED2.1 (VDD), LED3.1 (VDD), LED4.1 (VDD), LED5.1 (VDD), LED6.1 (VDD), LED7.1 (VDD), LED8.1 (VDD), LED9.1 (VDD), OLED1.2 (Pin_2)
Changed lines of the file:
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@@
 	)
 	(junction
-		(at 260.35 118.11)
-		(diameter 0)
-		(color 0 0 0 0)
-	)
-	(junction
 		(at 66.04 340.36)
 		(diameter 0)
@@
 	(wire
 		(pts
-			(xy 285.75 91.44) (xy 289.56 91.44)
-		)
-		(stroke
-			(width 0)
-			(type default)
-		)
-	)
-	(wire
-		(pts
 			(xy 87.63 252.73) (xy 111.76 252.73)
 		)
@@
 	(wire
 		(pts
+			(xy 283.21 105.41) (xy 287.02 105.41)
+		)
+		(stroke
+			(width 0)
+			(type default)
+		)
+	)
+	(wire
+		(pts
 			(xy 279.4 339.09) (xy 279.4 344.17)
 		)
@@
 	(wire
 		(pts
-			(xy 283.21 118.11) (xy 260.35 118.11)
-		)
-		(stroke
-			(width 0)
-			(type default)
-		)
-	)
-	(wire
-		(pts
 			(xy 181.61 321.31) (xy 181.61 293.37)
 		)
@@
 	(wire
 		(pts
-			(xy 260.35 41.91) (xy 260.35 44.45)
-		)
-		(stroke
-			(width 0)
-			(type default)
-		)
-	)
-	(wire
-		(pts
 			(xy 86.36 350.52) (xy 96.52 350.52)
 		)
@@
 	(wire
 		(pts
-			(xy 285.75 90.17) (xy 285.75 91.44)
-		)
-		(stroke
-			(width 0)
-			(type default)
-		)
-	)
-	(wire
-		(pts
 			(xy 129.54 349.25) (xy 129.54 321.31)
 		)
@@
 	(wire
 		(pts
-			(xy 283.21 105.41) (xy 283.21 118.11)
-		)
-		(stroke
-			(width 0)
-			(type default)
-		)
-	)
-	(wire
-		(pts
 			(xy 86.36 322.58) (xy 96.52 322.58)
 		)
@@
 	(wire
 		(pts
+			(xy 260.35 33.02) (xy 260.35 44.45)
+		)
+		(stroke
+			(width 0)
+			(type default)
+		)
+	)
+	(wire
+		(pts
 			(xy 262.89 321.31) (xy 262.89 311.15)
 		)
@@
 	(wire
 		(pts
-			(xy 283.21 90.17) (xy 285.75 90.17)
-		)
-		(stroke
-			(width 0)
-			(type default)
-		)
-	)
-	(wire
-		(pts
 			(xy 232.41 293.37) (xy 229.87 293.37)
 		)
@@
 	)
 	(symbol
+		(lib_id "dumbpad-eagle-import:GND")
+		(at 287.02 107.95 0)
+		(unit 1)
+		(exclude_from_sim no)
+		(in_bom yes)
+		(on_board yes)
+		(dnp no)
+		(property "Reference" "#GND02"
+			(at 287.02 107.95 0)
+			(effects
+				(font
+					(size 1.27 1.27)
+				)
+				(hide yes)
+			)
+		)
+		(property "Value" "GND"
+			(at 284.48 110.49 0)
+			(effects
+				(font
+					(size 1.778 1.5113)
+				)
+				(justify left bottom)
+			)
+		)
+		(property "Footprint" "dumbpad:"
+			(at 287.02 107.95 0)
+			(effects
+				(font
+					(size 1.27 1.27)
+				)
+				(hide yes)
+			)
+		)
+		(property "Datasheet" ""
+			(at 287.02 107.95 0)
+			(effects
+				(font
+					(size 1.27 1.27)
+				)
+				(hide yes)
+			)
+		)
+		(property "Description" ""
+			(at 287.02 107.95 0)
+			(effects
+				(font
+					(size 1.27 1.27)
+				)
+			)
+		)
+		(pin "1"
+		)
+		(instances
+			(project "17B06E-Macropad"
+				(path "/c58960d9-4cac-4036-ad2e-1aef26946dae"
+					(reference "#GND02")
+					(unit 1)
+				)
+			)
+		)
+	)
+	(symbol
 		(lib_id "Switch:SW_Push")
 		(at 101.6 266.7 0)
@@
 		(on_board yes)
 		(dnp no)
-		(fields_autoplaced yes)
 		(property "Reference" "OLED1"
-			(at 233.68 152.3999 0)
+			(at 233.68 151.384 0)
 			(effects
 				(font
@@
 		)
 		(property "Value" "I2C_OLED_0,91_Zoll_128X32"
-			(at 233.68 154.9399 0)
+			(at 233.68 153.67 0)
 			(effects
 				(font
@@
 			)
 		)
+		(property "I2C" "I²C1"
+			(at 233.68 156.464 0)
+			(effects
+				(font
+					(size 1.27 1.27)
+				)
+				(justify left)
+			)
+		)
 		(pin "4"
 		)
@@
 			)
 		)
-		(property "Value" "VCC"
+		(property "Value" "VCC +5V"
 			(at 106.68 20.32 0)
 			(effects
@@
 			)
 		)
-		(property "Value" "VCC"
+		(property "Value" "VCC +5V"
 			(at 218.186 152.4 0)
 			(effects
@@
 	)
 	(symbol
+		(lib_id "dumbpad-eagle-import:VCC")
+		(at 260.35 33.02 0)
+		(unit 1)
+		(exclude_from_sim no)
+		(in_bom yes)
+		(on_board yes)
+		(dnp no)
+		(property "Reference" "#SUPPLY03"
+			(at 260.35 33.02 0)
+			(effects
+				(font
+					(size 1.27 1.27)
+				)
+				(hide yes)
+			)
+		)
+		(property "Value" "VCC +5V"
+			(at 260.35 30.226 0)
+			(effects
+				(font
+					(size 1.778 1.5113)
+				)
+				(justify bottom)
+			)
+		)
+		(property "Footprint" "dumbpad:"
+			(at 260.35 33.02 0)
+			(effects
+				(font
+					(size 1.27 1.27)
+				)
+				(hide yes)
+			)
+		)
+		(property "Datasheet" ""
+			(at 260.35 33.02 0)
+			(effects
+				(font
+					(size 1.27 1.27)
+				)
+				(hide yes)
+			)
+		)
+		(property "Description" ""
+			(at 260.35 33.02 0)
+			(effects
+				(font
+					(size 1.27 1.27)
+				)
+			)
+		)
+		(pin "1"
+		)
+		(instances
+			(project "17B06E-Macropad"
+				(path "/c58960d9-4cac-4036-ad2e-1aef26946dae"
+					(reference "#SUPPLY03")
+					(unit 1)
+				)
+			)
+		)
+	)
+	(symbol
 		(lib_id "dumbpad-eagle-import:DIODEDO-1N4148")
 		(at 66.04 293.37 0)
@@
 					(unit 1)
 				)
-			)
-		)
-	)
-	(symbol
-		(lib_id "dumbpad-eagle-import:VCC")
-		(at 289.56 91.44 0)
-		(unit 1)
-		(exclude_from_sim no)
-		(in_bom yes)
-		(on_board yes)
-		(dnp no)
-		(property "Reference" "#SUPPLY02"
-			(at 289.56 91.44 0)
-			(effects
-				(font
-					(size 1.27 1.27)
-				)
-				(hide yes)
-			)
-		)
-		(property "Value" "VCC"
-			(at 289.56 88.646 0)
-			(effects
-				(font
-					(size 1.778 1.5113)
-				)
-				(justify bottom)
-			)
-		)
-		(property "Footprint" "dumbpad:"
-			(at 289.56 91.44 0)
-			(effects
-				(font
-					(size 1.27 1.27)
-				)
-				(hide yes)
-			)
-		)
-		(property "Datasheet" ""
-			(at 289.56 91.44 0)
-			(effects
-				(font
-					(size 1.27 1.27)
-				)
-				(hide yes)
-			)
-		)
-		(property "Description" ""
-			(at 289.56 91.44 0)
-			(effects
-				(font
-					(size 1.27 1.27)
-				)
-			)
-		)
-		(pin "1"
-		)
-		(instances
-			(project ""
-				(path "/c58960d9-4cac-4036-ad2e-1aef26946dae"
-					(reference "#SUPPLY02")
-					(unit 1)
-				)

Commit message: Various adjustments/improvements
Connections:
- net ENCODER_L5: no longer A1.31 (GPIO26_ADC0)
- net ENCODER_L1 renamed ENCODER_L1a
- net ENCODER_L2 renamed ENCODER_L2b
- net ENCODER_L3 renamed ENCODER_L3b
- net ENCODER_L4 renamed ENCODER_L4a
- net ENCODER_L6 renamed ENCODER_L6a
- net ENCODER_L7 renamed ENCODER_L7b
- net ENCODER_L8 renamed ENCODER_L8b
- net ENCODER_L9 renamed ENCODER_L9b
- new net ENCODER_L5b: A1.31 (GPIO26_ADC0)
Changed lines of the file:
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@@
 		)
 	)
-	(label "ENCODER_L6"
+	(label "ENCODER_L6a"
 		(at 224.79 105.41 0)
 		(effects
@@
 		)
 	)
-	(label "ENCODER_L4"
+	(label "ENCODER_L4a"
 		(at 287.02 97.79 0)
 		(effects
@@
 		)
 	)
-	(label "ENCODER_L3"
+	(label "ENCODER_L3b"
 		(at 22.86 298.45 0)
 		(effects
@@
 		)
 	)
-	(label "ENCODER_L1"
+	(label "ENCODER_L1a"
 		(at 24.13 238.76 0)
 		(effects
@@
 		)
 	)
-	(label "ENCODER_L4"
+	(label "ENCODER_L4a"
 		(at 24.13 325.12 0)
 		(effects
@@
 		)
 	)
-	(label "ENCODER_L7"
+	(label "ENCODER_L7b"
 		(at 307.34 242.57 0)
 		(effects
@@
 		)
 	)
-	(label "ENCODER_L7"
+	(label "ENCODER_L7b"
 		(at 224.79 102.87 0)
 		(effects
@@
 		)
 	)
-	(label "ENCODER_L8"
+	(label "ENCODER_L8b"
 		(at 307.34 298.45 0)
 		(effects
@@
 		)
 	)
-	(label "ENCODER_L9"
+	(label "ENCODER_L9b"
 		(at 307.34 349.25 0)
 		(effects
@@
 		)
 	)
-	(label "ENCODER_L8"
+	(label "ENCODER_L8b"
 		(at 224.79 100.33 0)
 		(effects
@@
 		)
 	)
-	(label "ENCODER_L5"
+	(label "ENCODER_L5b"
 		(at 287.02 95.25 0)
 		(effects
@@
 		)
 	)
-	(label "ENCODER_L3"
+	(label "ENCODER_L3b"
 		(at 287.02 100.33 0)
 		(effects
@@
 		)
 	)
-	(label "ENCODER_L2"
+	(label "ENCODER_L2b"
 		(at 224.79 69.85 0)
 		(effects
@@
 		)
 	)
-	(label "ENCODER_L9"
+	(label "ENCODER_L9b"
 		(at 224.79 97.79 0)
 		(effects
@@
 		)
 	)
-	(label "ENCODER_L6"
+	(label "ENCODER_L6a"
 		(at 307.34 237.49 0)
 		(effects
@@
 		)
 	)
-	(label "ENCODER_L1"
+	(label "ENCODER_L1a"
 		(at 224.79 72.39 0)
 		(effects
@@
 		)
 	)
-	(label "ENCODER_L2"
+	(label "ENCODER_L2b"
 		(at 24.13 243.84 0)
 		(effects

Commit message: Encoder better labeled as a/b in the schematic
Connections:
- net ENCODER_L5b is gone; now on net ENCODER3_b: A1.31 (GPIO26_ADC0)
- net ENCODER_L1a renamed ENCODER1u2_a
- net ENCODER_L2b renamed ENCODER1_b
- net ENCODER_L3b renamed ENCODER2_b
- net ENCODER_L4a renamed ENCODER3u6_a
- net ENCODER_L5 renamed ENCODER3_b
- net ENCODER_L6a renamed ENCODER4u5_a
- net ENCODER_L7b renamed ENCODER4_b
- net ENCODER_L8b renamed ENCODER5_b
- net ENCODER_L9b renamed ENCODER6_b
Changed lines of the file:
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@@
 	(wire
 		(pts
-			(xy 224.79 102.87) (xy 237.49 102.87)
+			(xy 223.52 102.87) (xy 237.49 102.87)
 		)
 		(stroke
@@
 	(wire
 		(pts
-			(xy 224.79 69.85) (xy 237.49 69.85)
+			(xy 223.52 69.85) (xy 237.49 69.85)
 		)
 		(stroke
@@
 	(wire
 		(pts
-			(xy 224.79 72.39) (xy 237.49 72.39)
+			(xy 223.52 72.39) (xy 237.49 72.39)
 		)
 		(stroke
@@
 	(wire
 		(pts
-			(xy 224.79 100.33) (xy 237.49 100.33)
+			(xy 223.52 100.33) (xy 237.49 100.33)
 		)
 		(stroke
@@
 	(wire
 		(pts
-			(xy 224.79 105.41) (xy 237.49 105.41)
+			(xy 223.52 105.41) (xy 237.49 105.41)
 		)
 		(stroke
@@
 	(wire
 		(pts
-			(xy 224.79 97.79) (xy 237.49 97.79)
+			(xy 223.52 97.79) (xy 237.49 97.79)
 		)
 		(stroke
@@
 		)
 	)
-	(label "ENCODER_L5"
+	(label "ENCODER3_b"
 		(at 24.13 330.2 0)
 		(effects
@@
 		)
 	)
-	(label "ENCODER_L6a"
-		(at 224.79 105.41 0)
+	(label "ENCODER4u5_a"
+		(at 223.52 105.41 0)
 		(effects
 			(font
@@
 		)
 	)
-	(label "ENCODER_L4a"
+	(label "ENCODER3u6_a"
 		(at 287.02 97.79 0)
 		(effects
@@
 		)
 	)
-	(label "ENCODER_L3b"
+	(label "ENCODER2_b"
 		(at 22.86 298.45 0)
 		(effects
@@
 		)
 	)
-	(label "ENCODER_L1a"
+	(label "ENCODER1u2_a"
 		(at 24.13 238.76 0)
 		(effects
@@
 		)
 	)
-	(label "ENCODER_L4a"
+	(label "ENCODER3u6_a"
 		(at 24.13 325.12 0)
 		(effects
@@
 		)
 	)
-	(label "ENCODER_L7b"
+	(label "ENCODER4_b"
 		(at 307.34 242.57 0)
 		(effects
@@
 		)
 	)
-	(label "ENCODER_L7b"
-		(at 224.79 102.87 0)
+	(label "ENCODER4_b"
+		(at 223.52 102.87 0)
 		(effects
 			(font
@@
 		)
 	)
-	(label "ENCODER_L8b"
+	(label "ENCODER5_b"
 		(at 307.34 298.45 0)
 		(effects
@@
 		)
 	)
-	(label "ENCODER_L9b"
+	(label "ENCODER6_b"
 		(at 307.34 349.25 0)
 		(effects
@@
 		)
 	)
-	(label "ENCODER_L8b"
-		(at 224.79 100.33 0)
-		(effects
-			(font
-				(size 1.2446 1.2446)
-			)
-			(justify left bottom)
-		)
-	)
-	(label "ENCODER_L5b"
+	(label "ENCODER5_b"
+		(at 223.52 100.33 0)
+		(effects
+			(font
+				(size 1.2446 1.2446)
+			)
+			(justify left bottom)
+		)
+	)
+	(label "ENCODER3_b"
 		(at 287.02 95.25 0)
 		(effects
@@
 		)
 	)
-	(label "ENCODER_L3b"
+	(label "ENCODER2_b"
 		(at 287.02 100.33 0)
 		(effects
@@
 		)
 	)
-	(label "ENCODER_L2b"
-		(at 224.79 69.85 0)
-		(effects
-			(font
-				(size 1.2446 1.2446)
-			)
-			(justify left bottom)
-		)
-	)
-	(label "ENCODER_L9b"
-		(at 224.79 97.79 0)
-		(effects
-			(font
-				(size 1.2446 1.2446)
-			)
-			(justify left bottom)
-		)
-	)
-	(label "ENCODER_L6a"
+	(label "ENCODER1_b"
+		(at 223.52 69.85 0)
+		(effects
+			(font
+				(size 1.2446 1.2446)
+			)
+			(justify left bottom)
+		)
+	)
+	(label "ENCODER6_b"
+		(at 223.52 97.79 0)
+		(effects
+			(font
+				(size 1.2446 1.2446)
+			)
+			(justify left bottom)
+		)
+	)
+	(label "ENCODER4u5_a"
 		(at 307.34 237.49 0)
 		(effects
@@
 		)
 	)
-	(label "ENCODER_L1a"
-		(at 224.79 72.39 0)
+	(label "ENCODER1u2_a"
+		(at 223.52 72.39 0)
 		(effects
 			(font
@@
 		)
 	)
-	(label "ENCODER_L2b"
+	(label "ENCODER1_b"
 		(at 24.13 243.84 0)
 		(effects

Commit message: various changes
holes changed, 
schematic correctly arranged,
and even more
Other:
- moved on the sheet: D1, D10, D12, D13, D15, D21, D22, D23, D24, D25, D26, D27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
