File: KiCad/17B06E-Macropad.kicad_pcb (KiCad board)
At the start: 2 copper layers, 128.8 x 102.8 mm, 72 parts, among them SW1 RotaryEncoder_Switch, SW2 RotaryEncoder_Switch, SW3 RotaryEncoder_Switch, SW4 RotaryEncoder_Switch, SW5 RotaryEncoder_Switch, SW6 RotaryEncoder_Switch

Commit message: URL to Codeberg
Repo migration
Other:
- board text added: "codeberg.org/Simon99de/17B06E-Macropad"
- board text removed: "github.com/Simon99de/17B06E-Macropad"
